File: hardware/analog_io.kicad_sch (KiCad schematic)
At the start: 0 parts

Commit message: block refactoring
Parts:
- added C8 (x2): 1uF, Capacitor_SMD:C_0603_1608Metric, symbol Device:C
- added D7 (x2), D8 (x2): D_SCHOTTKY_30V, Diode_SMD:D_SOD-123, symbol Device:D_Schottky_Small
- added J5: Conn_01x02/AIN, TerminalBlock:TerminalBlock_Altech_AK300-2_P5.00mm, symbol Connector_Generic:Conn_01x02
- added R19 (x2): 1M, Resistor_SMD:R_0603_1608Metric, symbol Device:R
- added R9 (x2): 100k, Resistor_SMD:R_0603_1608Metric, symbol Device:R
Connections:
- new net +3.3V: D7.1 (K), D7.1 (K)
- new net AIN1: C8.1, D7.2 (A), D8.1 (K), R19.1, R9.1
- new net AIN2: C8.1, D7.2 (A), D8.1 (K), R19.1, R9.1
- new net AIN_LINE1: J5.1 (Pin_1), R9.2
- new net AIN_LINE2: J5.2 (Pin_2), R9.2
- new net GND: C8.2, C8.2, D8.2 (A), D8.2 (A), R19.2, R19.2
