File: hardware/canbus.kicad_sch (KiCad schematic)
At the start: 26 parts, among them J601 Conn_01x04, U2 XL1509-3.3, U3 RCLAMP0524P-N, U501 SN65HVD230DR, U502 ADuM1201AR

Commit message: block refactoring
Parts:
- removed C4: 470uF/50V, Capacitor_SMD:C_0805_2012Metric, symbol Device:C
- removed C5: 4.7uF/50V, Capacitor_SMD:C_1206_3216Metric, symbol Device:C
- removed C504, C602, C604: 100nF, Capacitor_SMD:C_0402_1005Metric, symbol Device:C
- removed C6: 330uF, Capacitor_SMD:C_0402_1005Metric, symbol Device:C_Small
- removed D4, D6: B5819W, Diode_SMD:D_SOD-123, symbol Device:D_Schottky
- removed D5: SS24FL, Diode_SMD:D_SOD-123F, symbol Device:D_Schottky
- removed F2, F3, F4: ASMD1206-050, Fuse:Fuse_1206_3216Metric, symbol Device:Fuse
- removed J601: Conn_01x04, Connector_Phoenix_MC:PhoenixContact_MCV_1,5_4-G-3.81_1x04_P3.81mm_Vertical, symbol Connector_Generic:Conn_01x04
- removed JP1, JP2, JP601: SolderJumper_2_Open, SH-ESP32:SolderJumper-2_P1.3mm_Open_TrianglePad_Narrow, symbol Jumper:SolderJumper_2_Open
- removed L2: SMMS0650-470M, SH-ESP32:SMMS0650-1R0M, symbol Device:L
- removed NT1: NetTie_2, symbol Device:NetTie_2
- removed R213, R503: 10k, Resistor_SMD:R_0402_1005Metric, symbol Device:R_Small
- removed R601, R602: 240R, Resistor_SMD:R_0805_2012Metric, symbol Device:R
- removed U2: XL1509-3.3, Package_SO:SOP-8_3.9x4.9mm_P1.27mm, symbol SH-ESP32:XL1509-ADJE1
- removed U3: RCLAMP0524P-N, Package_DFN_QFN:Diodes_UDFN-10_1.0x2.5mm_P0.5mm, symbol SH-ESP32:RCLAMP0524P-N
- removed U501: SN65HVD230DR, Package_SO:SOIC-8_3.9x4.9mm_P1.27mm, symbol Interface_CAN_LIN:SN65HVD231
- removed U502: ADuM1201AR, Package_SO:SOIC-8_3.9x4.9mm_P1.27mm, symbol Isolator:ADuM1201AR
Connections:
- no-connect marks 3 -> 0
Other:
- note removed: "CAN Bus Connector"
- note removed: "CAN Isolated Power"
- note removed: "CAN Transceiver"
- note removed: "Jumper to connect CAN and PWR grounds"
- note removed: "Jumper to power global VIN from CAN bus"
- note removed: "Optional termination resistance for the bus"
- note removed: "Polarity & Surge Protection"
- note removed: "Rs provides slope control to limit EMI."
- note removed: "TODO - Replace with single opto isolated CAN tx ic"
- note removed: "TODO - size CAN signal fuses - check specs and pricing of TVS"
